File: hardware/0.1/samd21-pmod.kicad_pcb (KiCad board)
At the start: 2 copper layers, 40.6 x 40 mm, 29 parts, among them J1 USB_Type_C_2.0, J2 PMOD, J3 PWR, J4 PMOD, J5 SWD, SW1 SW_Push, U1 AP2112K-3.3, U3 ATSAMD21E17A-M, U4 W25Q32JVSSIQ

Commit message: tidy up routing
Parts:
- added REF**: Josh Details, josh-logos:josh-details, B.Cu at (146.0, 83.0)
Routing:
- net +3V3: track 139.8 -> 139.9 mm, vias 5 -> 4
- net GND: track 38.1 -> 38.2 mm, vias 74 -> 66
Other:
- board text added: "D0 | D4"
- board text added: "D1 | MOSI"
- board text added: "D2 | MISO"
- board text added: "D3 | SCK"
- board text added: "D5 | A2_RX"
- board text added: "D6 | A3"
- board text added: "RST"
- board text added: "SAMD21 PMOD"
- board text added: "SCL | A0"
- board text added: "SDA | A1_TX"
- board text removed: "RESET"
