File: hardware/0.1/samd21-pmod.kicad_sch (KiCad schematic)
At the start: 29 parts, among them J1 USB_Type_C_2.0, J2 PMOD, J3 PWR, J4 PMOD, J5 SWD, SW1 SW_Push, U1 AP2112K-3.3, U3 ATSAMD21E17A-M, U4 W25Q32JVSSIQ

Commit message: tidy up routing
Other:
- note added: "Dual PMOD"
Changed lines of the file:
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@@
     (stroke (width 0) (type solid) (color 0 0 0 0))
+  )
+  (text "Dual PMOD" (at 317.5 81.28 0)
+    (effects (font (size 2.54 2.54)) (justify left bottom))
   )
   (label "USB_D-" (at 67.31 82.55 180)
